Commit message: tool added

File: staubli_tx90_gazebo/urdf/tx90_macro.xacro (robot description, xacro)
@@ -66,4 +66,14 @@
     </actuator>
   </transmission>
+<!--   <transmission name="${prefix}tran7">
+    <robotNamespace>/${prefix}</robotNamespace>
+    <type>transmission_interface/SimpleTransmission</type>
+    <joint name="${prefix}joint_7">
+      <hardwareInterface>hardware_interface/PositionJointInterface</hardwareInterface>
+    </joint>
+    <actuator name="${prefix}motor7">
+      <mechanicalReduction>1</mechanicalReduction>
+    </actuator>
+  </transmission> -->
   <!-- end of transmission list -->
   <!-- Gazebo-specific link properties -->
@@ -96,4 +106,8 @@
     <turnGravityOff>true</turnGravityOff>
   </gazebo>
+  <gazebo reference="${prefix}link_7">
+    <material>Gazebo/Grey</material>
+    <turnGravityOff>true</turnGravityOff>
+  </gazebo>
   <!-- ros_control plugin -->
   <gazebo>

File: staubli_tx90_support/urdf/tx90_macro.xacro (robot description, xacro)
@@ -148,4 +148,26 @@
         <geometry>
           <mesh filename="package://staubli_tx90_support/meshes/tx90/collision/link_6.stl"/>
+        </geometry>
+      </collision>
+      <inertial>
+          <mass value="0.03098"/>
+          <origin xyz="-0.000243 0.050000 -0.006293" rpy="0.0 0.0 0.0"/>
+          <inertia ixx="0.000012" ixy="0.000000" ixz="0.000000"
+                                  iyy="0.000011" iyz="0.000000"
+                                                 izz="0.000022"/>
+      </inertial>
+    </link>
+    <link name="${prefix}link_7">
+      <visual>
+        <origin xyz="0 0 0" rpy="0 0 0"/>
+        <geometry>
+          <mesh filename="package://staubli_tx90_support/meshes/tx90/visual/link_5.stl"/>
+        </geometry>
+        <xacro:material_staubli_ral_grey_aluminium />
+      </visual>
+      <collision>
+        <origin xyz="0 0 0" rpy="0 0 0"/>
+        <geometry>
+          <mesh filename="package://staubli_tx90_support/meshes/tx90/collision/link_5.stl"/>
         </geometry>
       </collision>
@@ -210,4 +232,9 @@
       <dynamics damping="0.0" friction="0.0"/>
     </joint>
+    <joint name="${prefix}joint_7" type="fixed">
+      <origin xyz="0 0 0.100" rpy="0 0 0"/>
+      <parent link="${prefix}link_6"/>
+      <child link="${prefix}link_7"/>
+    </joint>
     <!-- ROS-Industrial 'base' frame: base_link to Staubli World Coordinates transform -->
     <link name="${prefix}base" />
@@ -221,5 +248,5 @@
     <joint name="${prefix}joint_6-flange" type="fixed">
       <origin xyz="0 0 0" rpy="0 ${radians(-90.0)} 0" />
-      <parent link="${prefix}link_6" />
+      <parent link="${prefix}link_7" />
       <child link="${prefix}flange" />
     </joint>
